Commit message: lab 3 no comments yet

File: urdf/robot.xacro (robot description, xacro)
@@ -1,37 +1,39 @@
 <?xml version='1.0'?>
 <robot name="robot" xmlns:xacro="http://www.ros.org/wiki/xacro">
-  <xacro:property name="camera_width" value="0.02"/>
+  <!-- Properties -->
+  <xacro:property name="camera_width"  value="0.02"/>
   <xacro:property name="camera_length" value="0.02"/>
   <xacro:property name="camera_height" value="0.01"/>
-  <xacro:property name="camera_mass" value="0.01"/>
-  <xacro:property name="chassis_width" value="0.15"/>
+  <xacro:property name="camera_mass"   value="0.01"/>
+  <xacro:property name="chassis_width"  value="0.15"/>
   <xacro:property name="chassis_length" value="0.2"/>
   <xacro:property name="chassis_height" value="0.05"/>
-  <xacro:property name="chassis_mass" value="0.5"/>
+  <xacro:property name="chassis_mass"   value="0.5"/>
   <xacro:property name="wheel_radius" value="0.04"/>
-  <xacro:property name="wheel_width" value="0.03"/>
-  <xacro:property name="wheel_mass" value="0.025"/>
+  <xacro:property name="wheel_width"  value="0.03"/>
+  <xacro:property name="wheel_mass"   value="0.025"/>
   <xacro:include filename="$(find enph353_ros_lab)/urdf/macros.xacro"/>
   <xacro:include filename="$(find enph353_ros_lab)/urdf/materials.xacro"/>
-  <link name='chassis'>
-    <xacro:box_inertial name="chassis" m="${chassis_mass}" x="${chassis_length}" y="${chassis_width}" z="${chassis_height}"/>
-    <collision name='chassis_collision'>
+  <!-- Chassis -->
+  <link name="chassis">
+    <xacro:box_inertial name="chassis" m="${chassis_mass}"
+                        x="${chassis_length}" y="${chassis_width}" z="${chassis_height}"/>
+    <collision name="chassis_collision">
       <geometry>
         <box size="${chassis_length} ${chassis_width} ${chassis_height}"/>
       </geometry>
     </collision>
-    <visual name='chassis_visual'>
-      <origin xyz="0 0 0" rpy=" 0 0 0"/>
+    <visual name="chassis_visual">
+      <origin xyz="0 0 0" rpy="0 0 0"/>
       <geometry>
         <box size="${chassis_length} ${chassis_width} ${chassis_height}"/>
       </geometry>
-      <material name="Cyan">
-        <color rgba="0 1.0 1.0 1.0"/>
-      </material>
+      <material name="Cyan"/>
     </visual>
   </link>
-  <link name='wheel_FR'>
+  <!-- Wheels -->
+  <link name="wheel_FR">
     <xacro:cylinder_inertial name="wheel_FR" m="${wheel_mass}" r="${wheel_radius}" h="${wheel_width}"/>
-    <collision name='wheel_FR_collision'>
+    <collision>
       <origin xyz="0 0 0" rpy="1.5708 0 0"/>
       <geometry>
@@ -39,5 +41,5 @@
       </geometry>
     </collision>
-    <visual name='wheel_FR_visual'>
+    <visual>
       <origin xyz="0 0 0" rpy="1.5708 0 0"/>
       <geometry>
@@ -46,7 +48,7 @@
     </visual>
   </link>
-  <link name='wheel_FL'>
+  <link name="wheel_FL">
     <xacro:cylinder_inertial name="wheel_FL" m="${wheel_mass}" r="${wheel_radius}" h="${wheel_width}"/>
-    <collision name='wheel_FL_collision'>
+    <collision>
       <origin xyz="0 0 0" rpy="1.5708 0 0"/>
       <geometry>
@@ -54,5 +56,5 @@
       </geometry>
     </collision>
-    <visual name='wheel_FL_visual'>
+    <visual>
       <origin xyz="0 0 0" rpy="1.5708 0 0"/>
       <geometry>
@@ -61,7 +63,7 @@
     </visual>
   </link>
-  <link name='wheel_RR'>
+  <link name="wheel_RR">
     <xacro:cylinder_inertial name="wheel_RR" m="${wheel_mass}" r="${wheel_radius}" h="${wheel_width}"/>
-    <collision name='wheel_RR_collision'>
+    <collision>
       <origin xyz="0 0 0" rpy="1.5708 0 0"/>
       <geometry>
@@ -69,5 +71,5 @@
       </geometry>
     </collision>
-    <visual name='wheel_RR_visual'>
+    <visual>
       <origin xyz="0 0 0" rpy="1.5708 0 0"/>
       <geometry>
@@ -76,7 +78,7 @@
     </visual>
   </link>
-  <link name='wheel_RL'>
+  <link name="wheel_RL">
     <xacro:cylinder_inertial name="wheel_RL" m="${wheel_mass}" r="${wheel_radius}" h="${wheel_width}"/>
-    <collision name='wheel_RL_collision'>
+    <collision>
       <origin xyz="0 0 0" rpy="1.5708 0 0"/>
       <geometry>
@@ -84,5 +86,5 @@
       </geometry>
     </collision>
-    <visual name='wheel_RL_visual'>
+    <visual>
       <origin xyz="0 0 0" rpy="1.5708 0 0"/>
       <geometry>
@@ -91,13 +93,14 @@
     </visual>
   </link>
-  <link name='camera_link'>
-    <xacro:box_inertial name="camera_link" m="${camera_mass}" x="${camera_width}" y="${camera_length}" z="${camera_height}"/>
-    <collision name='camera_link_collision'>
+  <!-- Camera -->
+  <link name="camera_link">
+    <xacro:box_inertial name="camera_link" m="${camera_mass}"
+                        x="${camera_width}" y="${camera_length}" z="${camera_height}"/>
+    <collision>
       <geometry>
         <box size="${camera_length} ${camera_width} ${camera_height}"/>
       </geometry>
     </collision>
-    <visual name='camera_link_visual'>
-      <origin xyz="0 0 0" rpy=" 0 0 0"/>
+    <visual>
       <geometry>
         <box size="${camera_length} ${camera_width} ${camera_height}"/>
@@ -105,9 +108,9 @@
     </visual>
   </link>
+  <!-- Joints -->
   <joint name="wheel_FR_joint" type="continuous">
     <parent link="chassis"/>
     <child link="wheel_FR"/>
-    <origin xyz="${chassis_length/2-wheel_radius} -${chassis_width/2+wheel_width/2} 0"
-            rpy="0 0 0"/>
+    <origin xyz="${chassis_length/2-wheel_radius} -${chassis_width/2+wheel_width/2} 0"/>
     <axis xyz="0 1 0"/>
   </joint>
@@ -115,6 +118,5 @@
     <parent link="chassis"/>
     <child link="wheel_FL"/>
-    <origin xyz="${chassis_length/2-wheel_radius} ${chassis_width/2+wheel_width/2} 0"
-            rpy="0 0 0"/>
+    <origin xyz="${chassis_length/2-wheel_radius} ${chassis_width/2+wheel_width/2} 0"/>
     <axis xyz="0 1 0"/>
   </joint>
@@ -122,6 +124,5 @@
     <parent link="chassis"/>
     <child link="wheel_RR"/>
-    <origin xyz="-${chassis_length/2-wheel_radius} -${chassis_width/2+wheel_width/2} 0"
-            rpy="0 0 0"/>
+    <origin xyz="-${chassis_length/2-wheel_radius} -${chassis_width/2+wheel_width/2} 0"/>
     <axis xyz="0 1 0"/>
   </joint>
@@ -129,6 +130,5 @@
     <parent link="chassis"/>
     <child link="wheel_RL"/>
-    <origin xyz="-${chassis_length/2-wheel_radius} ${chassis_width/2+wheel_width/2} 0"
-            rpy="0 0 0"/>
+    <origin xyz="-${chassis_length/2-wheel_radius} ${chassis_width/2+wheel_width/2} 0"/>
     <axis xyz="0 1 0"/>
   </joint>
@@ -138,21 +138,58 @@
     <origin xyz="${chassis_length/2} 0 ${chassis_height/2+camera_height/2}"/>
   </joint>
-  <gazebo reference="chassis">
-    <material>Gazebo/Orange</material>
+  <!-- Gazebo Materials -->
+  <gazebo reference="chassis"><material>Gazebo/Orange</material></gazebo>
+  <gazebo reference="camera_link"><material>Gazebo/Blue</material></gazebo>
+  <gazebo reference="wheel_FL"><material>Gazebo/Yellow</material></gazebo>
+  <gazebo reference="wheel_FR"><material>Gazebo/Yellow</material></gazebo>
+  <gazebo reference="wheel_RL"><material>Gazebo/Yellow</material></gazebo>
+  <gazebo reference="wheel_RR"><material>Gazebo/Yellow</material></gazebo>
+  <!-- Skid Steer Plugin -->
+  <gazebo>
+    <plugin name="skid_steer_drive_controller" filename="libgazebo_ros_skid_steer_drive.so">
+      <ros>
+        <namespace>/</namespace>
+        <remapping>cmd_vel:=cmd_vel</remapping>
+        <remapping>odom:=odom</remapping>
+      </ros>
+      <updateRate>100.0</updateRate>
+      <leftFrontJoint>wheel_FL_joint</leftFrontJoint>
+      <rightFrontJoint>wheel_FR_joint</rightFrontJoint>
+      <leftRearJoint>wheel_RL_joint</leftRearJoint>
+      <rightRearJoint>wheel_RR_joint</rightRearJoint>
+      <wheelSeparation>${chassis_width}</wheelSeparation>
+      <wheelDiameter>${2*wheel_radius}</wheelDiameter>
+      <odomFrame>odom</odomFrame>
+      <robotBaseFrame>chassis</robotBaseFrame>
+      <publishOdom>true</publishOdom>
+      <publishTf>true</publishTf>
+    </plugin>
   </gazebo>
+  <!-- Camera Sensor -->
   <gazebo reference="camera_link">
-    <material>Gazebo/Blue</material>
-  </gazebo>
-  <gazebo reference="wheel_FL">
-    <material>Gazebo/Yellow</material>
-  </gazebo>
-  <gazebo reference="wheel_FR">
-    <material>Gazebo/Yellow</material>
-  </gazebo>
-  <gazebo reference="wheel_RL">
-    <material>Gazebo/Yellow</material>
-  </gazebo>
-  <gazebo reference="wheel_RR">
-    <material>Gazebo/Yellow</material>
+    <sensor type="camera" name="camera_sensor">
+      <pose>0 0 0 0.0 0.785 0.0</pose>
+      <update_rate>30</update_rate>
+      <camera>
+        <horizontal_fov>1.047</horizontal_fov> <!-- ~60 deg -->
+        <image>
+          <width>640</width>
+          <height>480</height>
+          <format>R8G8B8</format>
+        </image>
+        <clip>
+          <near>0.02</near>
+          <far>5</far>
+        </clip>
+      </camera>
+      <plugin name="camera_controller" filename="libgazebo_ros_camera.so">
+        <ros>
+          <namespace>/</namespace>
+          <remapping>image_raw:=/camera/image_raw</remapping>
+          <remapping>camera_info:=/camera/camera_info</remapping>
+        </ros>
+        <frameName>camera_link</frameName>
+      </plugin>
+    </sensor>
   </gazebo>
 </robot>
